File: hardware/actuator-node/actuator-node.kicad_sch (KiCad schematic)
At the start: 53 parts, among them J1 PHASES, J2 CAN IN, J3 CAN EXT, J4 19V IN, J5 SWD, J6 ENCODER, J7 NTC, M1 SimpleFOC Mini, U1 STM32G431CBT6, U2 SN65HVD230, U4 INA240A1D, U5 INA240A1D, U6 AMS1117-3.3, Y1 8 MHz

Commit message: Rebuild both boards from the real driver module, grouped by function
The vendor's EasyEDA export of the driver module arrived, so its footprint is
now measured rather than guessed: 17 pins and four mounting holes over
22.6 x 18.2 mm, read from vendor/simplefoc_stepmini.json at build time.

The export also settles three things that were open, and raises one:

- The module's 3V3 pin is a supply input. Its nSLEEP and nRESET pull-ups hang
  off it and there is no regulator on the board, so leaving it open would have
  left the driver possibly held in reset. It is now wired to the 3.3 V rail.
- The header's enable pin sits behind a series resistor into the driver's EN,
  so the kill line drives it directly and nSLEEP/nRESET need no connection.
- nFAULT is brought out with its own pull-up, so it now goes to PB4.
- The export shows a quad half-bridge - IN1-IN4 and OUT1-OUT4 - not the
  three-in/three-out DRV8313 the build console names. A 3-phase motor uses
  three of the four channels, so it works, but it is not the specified part.
  Flagged in the actuator README rather than silently accepted.

Placement is now by functional block. Each block keeps its own passives, and
parts with an electrical reason to hug another are placed against it and
checked: the crystal is held within 12 mm of the MCU and its load caps within
9 mm of it, which the previous layout failed at 32 mm. Microphone spacing is
pinned at exactly 130 mm and verified. Both boards are larger - the node goes
to 70 x 60 and the base to 170 x 100 - which is what buys room to group and
still route by hand.

Indicators added on both boards, using the XL-3216SURC red 1206 that is on
hand. Series resistors are sized for its 2.4 V forward drop rather than left at
a default: 220 R on 3.3 V rails, 470 R on the 5 V one.

check.py grew to match: it now verifies group membership, pinned positions and
proximity constraints alongside the netlist, and each project carries a
colour-coded placement.svg.

Co-Authored-By: Claud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
Parts:
- added D2: XL-3216SURC red, LED_SMD:LED_1206_3216Metric, symbol Device:LED
- added R14: 220R, Resistor_SMD:R_1206_3216Metric, symbol Device:R
- D1: value red -> XL-3216SURC red
- R13: value 120R -> 220R
Connections:
- net +19V: now also M1.13 (VM); no longer M1.5 (VIN)
- net +3V3: now also M1.11 (3V3), D2.2 (A)
- net DRV_EN: now also M1.5 (EN); no longer M1.4 (EN)
- net GND: now also M1.10 (GND), M1.12 (GND), R14.2
- net PH_A_DRV: now also M1.14 (OUT1); no longer M1.7 (OUTA)
- net PH_B_DRV: now also M1.15 (OUT2); no longer M1.8 (OUTB)
- net PH_C: now also M1.16 (OUT3); no longer M1.9 (OUTC)
- net DRV_nFAULT: now reaches U1.41 (PB4)
- net DRV_nFAULT: now also M1.7 (nFAULT)
- new net PWR_LED_K: D2.1 (K), R14.1
Other:
- moved on the sheet: J1, J2, J3, J4, J5, J6, J7, JP1, JP2, JP3, JP4, R1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

Commit message: Rebuild the driver module around the real SimpleFOC Mini v1.0
The EasyEDA export the footprint was generated from was a different product:
a "step mini" quad half-bridge with IN1-IN4 and four outputs, where the board
on the bench is a SimpleFOC Mini v1.0 (DRV8313, three phases, dated 04/22).
The generated footprint carried phantom IN4/OUT4 pins, the wrong row order and
the wrong geometry, and would not have populated.

Everything now comes from the v1.0 exports. The PCB export gives pad geometry;
the schematic export resolves that PCB's anonymous U1_nn nets to real signals
and is what settled the important question below. Both step-mini exports are
removed.

Fixes a real bug this uncovered. The module's 3V3 header pin is DRV8313 pin 15,
V3P3OUT - an internal regulator output, not a supply input as previously
assumed. It had been wired to the carrier's 3.3 V rail, which would have
connected the AMS1117's output to the module's own regulator. It is now left
open, and check.py fails the build if it reappears on any net. That same
regulator feeds the module's nSlp/nRes/nFlt pull-ups, which is why those three
need no connection to idle in the running state.

The module's reference becomes A1 rather than M1, so its pins can carry the
silkscreen names M1/M2/M3 without ("M1", "M1") appearing in the netlist.

Two generator fixes fell out of the rebuild:

- simplefoc_from_json() now reads pads nested inside LIB entries, because on
  this board the headers are placed as components - only 6 of the 19 pads are
  top-level shapes - while filtering to the HDR-* components so the driver IC's
  own 29 pads stay out.
- Proximity placement follows each chain depth-first and ranks candidates by
  distance to the target's courtyard rather than to its origin. Breadth-first
  ranking by origin put a crystal load cap 3.8 mm clear of a crystal whose
  courtyard is 20 mm wide; both caps now sit inside 2 mm. check.py measures the
  same way, edge to edge, since centre-to-centre was mostly mea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
Parts:
- removed M1: SimpleFOC Mini, juno:SimpleFOC_Mini_Socket, symbol juno:SimpleFOC_Mini
- added A1: SimpleFOC Mini v1.0, juno:SimpleFOC_Mini_Socket, symbol juno:SimpleFOC_Mini
Connections:
- net +19V: now also A1.12 (VM)
- net DRV_EN: now also A1.1 (EN)
- net DRV_nFAULT: now also A1.6 (nFlt)
- net GND: now also A1.11 (GND), A1.5 (GND), A1.9 (GND)
- net PH_A_DRV: now also A1.13 (M1)
- net PH_B_DRV: now also A1.14 (M2)
- net PH_C: now also A1.15 (M3)
- net PWM_A: now also A1.4 (IN1)
- net PWM_B: now also A1.3 (IN2)
- net PWM_C: now also A1.2 (IN3)
Other:
- moved on the sheet: C1, C10, C11, C12, C13, C14, C15, C16, C17, C18, C19, C2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

Commit message: Rebuild the BOM around parts on hand, and target Lion Circuits
Every passive and semiconductor in both boards is now a part that is actually
on the shelf, with docs/parts.md recording the reconciliation. Four
substitutions were needed:

- LED series resistors move from 220R/470R, which are not stocked, to 120R on
  the 3.3 V rails (7.5 mA) and 1k on the brain's 5 V rail (2.6 mA, where 120R
  would exceed the LED's 20 mA rating).
- The kill-line gate series resistor moves from 100R to 120R, immaterial here.
- The reverse-polarity FET becomes the AO3481 that is actually on hand; KiCad
  has no symbol for it, so the projects use AO3401A, the same family and the
  same G/S/D pinout.
- The 10 V zener clamping that FET's gate is not stocked, so the gate is
  divided rather than clamped: 100k source-to-gate and 100k gate-to-ground put
  Vgs at about -9.5 V, which enhances the FET hard and stays well inside its
  rating. Two resistors that are stocked, replacing one part that is not.

Two items have no substitute and must be ordered: 30 mR shunts, without which
there is no current sensing, and an N-channel MOSFET for the kill line, since
the AO3481 on hand is P-channel and cannot pull the EN bus down. The kill line
is the one circuit that should not be improvised.

Also notes that the CD43 inductor supplied with the transceivers has no place
in either board, and why the one plausible use - an LC filter on the node's
5 V input - would resonate at about 28 kHz, right on top of the motor PWM.

For fabrication, the boards now carry plot settings that emit Protel-style
gerber extensions, matching the sample set from Lion Circuits, with the X2
attributes off so the output is plain RS-274X. docs/fabrication.md records
their file naming and the design rules used, and is explicit that their
capability page could not be reached from here, so those rules are a
conservative set rather than a reading of their spec sheet.

Co-Authored-By: Claude Opus 5 <noreply@anthropic.com>
Claude-Sess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
Parts:
- R13, R14: value 220R -> 120R
Changed lines of the file:
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@@
 			)
 		)
-		(property "Value" "220R"
+		(property "Value" "120R"
 			(at 218.44 187.96 0)
 			(effects
@@
 			)
 		)
-		(property "Value" "220R"
+		(property "Value" "120R"
 			(at 251.46 187.96 0)
 			(effects
@@
 		(on_board yes)
 		(dnp no)
-		(property "Reference" "#PWR818"
+		(property "Reference" "#PWR104"
 			(at 30 295.48 0)
 			(effects
@@
 			(project "actuator-node"
 				(path "/f591a9c0-9da4-4a37-a7ce-2a93192dc18f"
-					(reference "#PWR818")
+					(reference "#PWR104")
 					(unit 1)
 				)
@@
 		(on_board yes)
 		(dnp no)
-		(property "Reference" "#FLG818"
+		(property "Reference" "#FLG104"
 			(at 42.7 295.48 0)
 			(effects
@@
 			(project "actuator-node"
 				(path "/f591a9c0-9da4-4a37-a7ce-2a93192dc18f"
-					(reference "#FLG818")
+					(reference "#FLG104")
 					(unit 1)
 				)
@@
 		(on_board yes)
 		(dnp no)
-		(property "Reference" "#PWR366"
+		(property "Reference" "#PWR438"
 			(at 68.1 295.48 0)
 			(effects
@@
 			(project "actuator-node"
 				(path "/f591a9c0-9da4-4a37-a7ce-2a93192dc18f"
-					(reference "#PWR366")
+					(reference "#PWR438")
 					(unit 1)
 				)
@@
 		(on_board yes)
 		(dnp no)
-		(property "Reference" "#FLG366"
+		(property "Reference" "#FLG438"
 			(at 80.8 295.48 0)
 			(effects
@@
 			(project "actuator-node"
 				(path "/f591a9c0-9da4-4a37-a7ce-2a93192dc18f"
-					(reference "#FLG366")
+					(reference "#FLG438")
 					(unit 1)
 				)
@@
 		(on_board yes)
 		(dnp no)
-		(property "Reference" "#PWR234"
+		(property "Reference" "#PWR193"
 			(at 106.2 295.48 0)
 			(effects
@@
 			(project "actuator-node"
 				(path "/f591a9c0-9da4-4a37-a7ce-2a93192dc18f"
-					(reference "#PWR234")
+					(reference "#PWR193")
 					(unit 1)
 				)
@@
 		(on_board yes)
 		(dnp no)
-		(property "Reference" "#FLG234"
+		(property "Reference" "#FLG193"
 			(at 118.9 295.48 0)
 			(effects
@@
 			(project "actuator-node"
 				(path "/f591a9c0-9da4-4a37-a7ce-2a93192dc18f"
-					(reference "#FLG234")
+					(reference "#FLG193")
 					(unit 1)
 				)
@@
 		(on_board yes)
 		(dnp no)
-		(property "Reference" "#PWR542"
+		(property "Reference" "#PWR288"
 			(at 144.3 295.48 0)
 			(effects
@@
 			(project "actuator-node"
 				(path "/f591a9c0-9da4-4a37-a7ce-2a93192dc18f"
-					(reference "#PWR542")
+					(reference "#PWR288")
 					(unit 1)
 				)
@@
 		(on_board yes)
 		(dnp no)
-		(property "Reference" "#FLG542"
+		(property "Reference" "#FLG288"
 			(at 157 295.48 0)
 			(effects
@@
 			(project "actuator-node"
 				(path "/f591a9c0-9da4-4a37-a7ce-2a93192dc18f"
-					(reference "#FLG542")
-					(unit 1)
-				)
+					(reference "#FLG288")
+					(unit 1)
+				)

Commit message: Add an SPI header, floorplan the node, and render assembly views
SPI1 is added as J8, a 1x6 header carrying 3V3, GND, SCK, MISO, MOSI and CS on
PA4-PA7. Those four pins were entirely unused, so an upgrade to an SPI encoder
(AS5047P, MA730, TLE5012B) or an SPI-configured driver costs a header and no
re-assignment. SPI2 would have collided with the driver EN and the node-ID
jumpers, SPI3 with the driver fault line.

Connectors are now pinned to the perimeter on three rules: the two CAN
connectors face each other on opposite edges, since they are a daisy chain;
everything running to the motor - phases, encoder, stator thermistor and the
SPI header - leaves together on one edge as a single loom; and nothing sits in
the interior.

That squeezed the middle enough that auto-placement put the crystal 15 mm from
the MCU and a shunt 16 mm from its amplifier, so the parts that decide the
floorplan are placed by hand: driver socket and its bulk cap, MCU, crystal, and
each shunt beside its own INA240. The Kelvin tap has to land on the shunt's end
caps - at 30 mOhm, 20 mm of copper is a five percent error.

tools/render.py draws the board to SVG from the .kicad_pcb, with no new
dependencies: top assembly with dimensions, mirrored bottom, copper, and a
detail on the driver and MCU. It draws whatever copper is in the file, so the
same views show traces once the board is routed - today it reports zero and
says so on the copper view rather than looking merely empty.

Co-Authored-By: Claude Opus 5 <noreply@anthropic.com>
Claude-Session: https://claude.ai/code/session_011qFNDvbo1RnNn3sy9mr9bh
Parts:
- added J8: SPI, Connector_PinHeader_2.54mm:PinHeader_1x06_P2.54mm_Vertical, symbol Connector_Generic:Conn_01x06
Connections:
- net +3V3: now also J8.1 (Pin_1)
- net GND: now also J8.2 (Pin_2)
- net SPI_CS: now reaches U1.12 (PA4)
- net SPI_CS: now also J8.6 (Pin_6)
- net SPI_SCK: now reaches U1.13 (PA5)
- net SPI_SCK: now also J8.3 (Pin_3)
- net SPI_MISO: now reaches U1.14 (PA6)
- net SPI_MISO: now also J8.4 (Pin_4)
- net SPI_MOSI: now reaches U1.15 (PA7)
- net SPI_MOSI: now also J8.5 (Pin_5)
Other:
- moved on the sheet: JP1, JP2, JP3, JP4, R1, R10, R12, R13, R14, R2, R3, R4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

Commit message: Lay the node out around right-angle connectors, and spec what it can do
The connector order is all right-angle JST: 3-pin XH, 5-pin XH and 2-pin VH,
with no 2-pin XH at all. A right-angle body opens toward +Y at 0 degrees, so
the rotation is what points a cable off the board, and the placer had no
concept of rotation - it put J2 through the crystal and pushed J1 and J7 past
the outline.

kigen.rotate_boxes turns a footprint's courtyard with it; pinned entries now
take an optional third element; check.py rotates the library courtyard before
testing overlap and outline, and verifies the angle as well as the position.

Floorplan, following the three placement rules:
  - CAN on opposite edges, J2 left and J3 right
  - the whole motor loom on the bottom edge: phases, NTC, encoder, SPI
  - power and SWD on the top
All eight ports are on the perimeter, none closer than 1.1 mm to an edge.

Four things the auto-placer got wrong and are now pinned:
  - U6 sat under the driver module, stacking the LDO's heat under the bridge's
  - R7 sat on A1's exact origin; it belongs under the module, but deliberately
    placed clear of every pad rather than by accident
  - both crystal load caps sat at one end of a 20 mm hand-solder footprint,
    leaving one of them 22 mm from its terminal
  - the node-ID pull-ups were stranded 13 mm from their jumpers

Vbus divider R4 4k7 -> 10k. 100 k / 4k7 read 19 V as 0.85 V, a quarter of the
ADC span. 100 k / 10 k reads 1.73 V and clips at 36 V.

Two renderer bugs, both only visible once something was rotated or mirrored:
  - pad angles were being summed with the footprint angle, but KiCad stores a
    pad's angle absolutely
  - the mirror reflected about the origin rather than the view box, and the
    substrate rect took its min in board space instead of screen space, so the
    bottom view sat 13 mm left and grew a slab off the far edge

New docs:
  - docs/capabilities.md - bus range, torque and current resolution, loop
    rates, CAN bandwidth a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
Parts:
- J1: footprint Connector_JST:JST_XH_B3B-XH-A_1x03_P2.50mm_Vertical -> Connector_JST:JST_XH_S3B-XH-A_1x03_P2.50mm_Horizontal
- J2, J3: footprint Connector_JST:JST_XH_B5B-XH-AM_1x05_P2.50mm_Vertical -> Connector_JST:JST_XH_S5B-XH-A_1x05_P2.50mm_Horizontal
- J4: footprint Connector_JST:JST_VH_B2P-VH_1x02_P3.96mm_Vertical -> Connector_JST:JST_VH_S2P-VH_1x02_P3.96mm_Horizontal
- J7: footprint Connector_JST:JST_XH_B2B-XH-A_1x02_P2.50mm_Vertical -> Connector_JST:JST_XH_S3B-XH-A_1x03_P2.50mm_Horizontal; symbol Connector_Generic:Conn_01x02 -> Connector_Generic:Conn_01x03
- R4: value 4k7 -> 10k
Connections:
- net GND: now also J7.3 (Pin_3)
Changed lines of the file:
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@@
 	(wire
 		(pts
+			(xy 149.86 134.62) (xy 147.32 134.62)
+		)
+		(stroke
+			(width 0)
+			(type default)
+		)
+	)
+	(wire
+		(pts
 			(xy 182.88 129.54) (xy 180.34 129.54)
 		)
@@
 		)
 	)
+	(label "GND"
+		(at 147.32 134.62 180)
+		(effects
+			(font
+				(size 1.27 1.27)
+			)
+			(justify right bottom)
+		)
+	)
 	(label "+3V3"
 		(at 180.34 129.54 180)
@@
 			)
 		)
-		(property "Footprint" "Connector_JST:JST_XH_B3B-XH-A_1x03_P2.50mm_Vertical"
+		(property "Footprint" "Connector_JST:JST_XH_S3B-XH-A_1x03_P2.50mm_Horizontal"
 			(at 441.96 91.44 0)
 			(effects
@@
 			)
 		)
-		(property "Footprint" "Connector_JST:JST_XH_B5B-XH-AM_1x05_P2.50mm_Vertical"
+		(property "Footprint" "Connector_JST:JST_XH_S5B-XH-A_1x05_P2.50mm_Horizontal"
 			(at 477.52 93.98 0)
 			(effects
@@
 			)
 		)
-		(property "Footprint" "Connector_JST:JST_XH_B5B-XH-AM_1x05_P2.50mm_Vertical"
+		(property "Footprint" "Connector_JST:JST_XH_S5B-XH-A_1x05_P2.50mm_Horizontal"
 			(at 510.54 93.98 0)
 			(effects
@@
 			)
 		)
-		(property "Footprint" "Connector_JST:JST_VH_B2P-VH_1x02_P3.96mm_Vertical"
+		(property "Footprint" "Connector_JST:JST_VH_S2P-VH_1x02_P3.96mm_Horizontal"
 			(at 53.34 129.54 0)
 			(effects
@@
 	)
 	(symbol
-		(lib_id "Connector_Generic:Conn_01x02")
-		(at 154.94 129.54 0)
+		(lib_id "Connector_Generic:Conn_01x03")
+		(at 154.94 132.08 0)
 		(unit 1)
 		(exclude_from_sim no)
@@
 		(dnp no)
 		(property "Reference" "J7"
-			(at 154.94 116.84 0)
+			(at 154.94 119.38 0)
 			(effects
 				(font
@@
 		)
 		(property "Value" "NTC"
-			(at 154.94 142.24 0)
+			(at 154.94 144.78 0)
 			(effects
 				(font
@@
 			)
 		)
-		(property "Footprint" "Connector_JST:JST_XH_B2B-XH-A_1x02_P2.50mm_Vertical"
-			(at 154.94 129.54 0)
+		(property "Footprint" "Connector_JST:JST_XH_S3B-XH-A_1x03_P2.50mm_Horizontal"
+			(at 154.94 132.08 0)
 			(effects
 				(font
@@
 		)
 		(property "Datasheet" "~"
-			(at 154.94 129.54 0)
+			(at 154.94 132.08 0)
 			(effects
 				(font
@@
 		(pin "2"
 		)
+		(pin "3"
+		)
 		(instances
 			(project "actuator-node"
@@
 			)
 		)
-		(property "Value" "4k7"
+		(property "Value" "10k"
 			(at 487.68 147.32 0)
 			(effects
@@
 		(on_board yes)
 		(dnp no)
-		(property "Reference" "#PWR779"
+		(property "Reference" "#PWR620"
 			(at 30 305.64 0)
 			(effects
@@
 			(project "actuator-node"
 				(path "/f591a9c0-9da4-4a37-a7ce-2a93192dc18f"
-					(reference "#PWR779")
+					(reference "#PWR620")
 					(unit 1)
 				)
@@
 		(on_board yes)
 		(dnp no)
-		(property "Reference" "#FLG779"
+		(property "Reference" "#FLG620"
 			(at 42.7 305.64 0)
 			(effects
@@
 			(project "actuator-node"
 				(path "/f591a9c0-9da4-4a37-a7ce-2a93192dc18f"
-					(reference "#FLG779")
+					(reference "#FLG620")
 					(unit 1)
 				)
@@
 		(on_board yes)
 		(dnp no)
-		(property "Reference" "#PWR138"
+		(property "Reference" "#PWR687"
 			(at 68.1 305.64 0)
 			(effects
@@
 			(project "actuator-node"
 				(path "/f591a9c0-9da4-4a37-a7ce-2a93192dc18f"
-					(reference "#PWR138")
+					(reference "#PWR687")
 					(unit 1)
 				)
@@
 		(on_board yes)
 		(dnp no)
-		(property "Reference" "#FLG138"
+		(property "Reference" "#FLG687"
 			(at 80.8 305.64 0)
 			(effects
@@
 			(project "actuator-node"
 				(path "/f591a9c0-9da4-4a37-a7ce-2a93192dc18f"
-					(reference "#FLG138")
+					(reference "#FLG687")
 					(unit 1)
 				)
@@
 		(on_board yes)
 		(dnp no)
-		(property "Reference" "#PWR816"
+		(property "Reference" "#PWR397"
 			(at 106.2 305.64 0)
 			(effects
@@
 			(project "actuator-node"
 				(path "/f591a9c0-9da4-4a37-a7ce-2a93192dc18f"
-					(reference "#PWR816")
+					(reference "#PWR397")
 					(unit 1)
 				)
@@
 		(on_board yes)
 		(dnp no)
-		(property "Reference" "#FLG816"
+		(property "Reference" "#FLG397"
 			(at 118.9 305.64 0)
 			(effects
@@
 			(project "actuator-node"
 				(path "/f591a9c0-9da4-4a37-a7ce-2a93192dc18f"
-					(reference "#FLG816")
+					(reference "#FLG397")
 					(unit 1)
 				)
@@
 		(on_board yes)
 		(dnp no)
-		(property "Reference" "#PWR409"
+		(property "Reference" "#PWR291"
 			(at 144.3 305.64 0)
 			(effects
@@
 			(project "actuator-node"
 				(path "/f591a9c0-9da4-4a37-a7ce-2a93192dc18f"
-					(reference "#PWR409")
+					(reference "#PWR291")
 					(unit 1)
 				)
@@
 		(on_board yes)
 		(dnp no)
-		(property "Reference" "#FLG409"
+		(property "Reference" "#FLG291"
 			(at 157 305.64 0)
 			(effects
@@
 			(project "actuator-node"
 				(path "/f591a9c0-9da4-4a37-a7ce-2a93192dc18f"
-					(reference "#FLG409")
+					(reference "#FLG291")
 					(unit 1)
 				)
